File: boost_converter.kicad_sch (KiCad schematic)
At the start: 9 parts, among them Q1 DMG3404L

Commit message: assigned footprints
Parts:
- added J3: Conn_01x04, Connector_PinHeader_2.54mm:PinHeader_1x04_P2.54mm_Vertical, symbol Connector_Generic:Conn_01x04
- added R11: 30.1k, Resistor_SMD:R_0603_1608Metric_Pad0.98x0.95mm_HandSolder, symbol Device:R
- added R12, R15: 10k, Resistor_SMD:R_0603_1608Metric_Pad0.98x0.95mm_HandSolder, symbol Device:R
- C18: now not fitted
- L1: footprint (none) -> Inductor_SMD:L_Bourns_SRR1260
Connections:
- net GND: now also J3.3 (Pin_3), R12.2
- net +12V: now reaches C1.1, C7.1, C8.1, D1.1 (K)
- net +12V: now also J3.1 (Pin_1), R11.1
- net VSYS: now reaches C18.1, C19.1, L1.1
- net I_SNS: now reaches R1.2
- net I_SNS: now also J3.2 (Pin_2)
- net GATE: now reaches Q1.1 (G)
- new net +3V3: R15.2
- new net Ambient_Light: J3.4 (Pin_4), R15.1
- new net U_SNS: R11.2, R12.1
Other:
- note added: "1.6mA /LSB"
- note added: "3.2mV/lsb"
- moved on the sheet: R1

Commit message: Layout begonnen
Parts:
- L1: footprint Inductor_SMD:L_Bourns_SRR1260 -> Inductor_SMD:L_Bourns_SRR1260_handsolder
Changed lines of the file:
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@@
 			)
 		)
-		(property "Footprint" "Inductor_SMD:L_Bourns_SRR1260"
+		(property "Footprint" "Inductor_SMD:L_Bourns_SRR1260_handsolder"
 			(at 123.19 76.2 0)
 			(effects

Commit message: marked unused capaacitors as not placed. Pull down on gate channel
Parts:
- added R16: 10k, Resistor_SMD:R_0603_1608Metric_Pad0.98x0.95mm_HandSolder, symbol Device:R
Connections:
- net GATE: now also R16.1
- net GND: now also R16.2
Changed lines of the file:
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@@
+	)
+	(junction
+		(at 127 86.36)
+		(diameter 0)
+		(color 0 0 0 0)
 	)
 	(junction
@@
 	(wire
 		(pts
+			(xy 127 93.98) (xy 127 95.25)
+		)
+		(stroke
+			(width 0)
+			(type default)
+		)
+	)
+	(wire
+		(pts
 			(xy 166.37 90.17) (xy 166.37 96.52)
 		)
@@
 		(pts
 			(xy 219.71 114.3) (xy 215.9 114.3)
+		)
+		(stroke
+			(width 0)
+			(type default)
+		)
+	)
+	(wire
+		(pts
+			(xy 124.46 86.36) (xy 127 86.36)
 		)
 		(stroke
@@
 	(global_label "GATE"
 		(shape input)
-		(at 127 86.36 180)
+		(at 124.46 86.36 180)
 		(fields_autoplaced yes)
 		(effects
@@
 		)
 		(property "Intersheetrefs" "${INTERSHEET_REFS}"
-			(at 119.5396 86.36 0)
+			(at 116.9996 86.36 0)
 			(effects
 				(font
@@
 	)
 	(symbol
+		(lib_id "power:GND")
+		(at 127 95.25 0)
+		(unit 1)
+		(exclude_from_sim no)
+		(in_bom yes)
+		(on_board yes)
+		(dnp no)
+		(fields_autoplaced yes)
+		(property "Reference" "#PWR045"
+			(at 127 101.6 0)
+			(effects
+				(font
+					(size 1.27 1.27)
+				)
+				(hide yes)
+			)
+		)
+		(property "Value" "GND"
+			(at 127 100.33 0)
+			(effects
+				(font
+					(size 1.27 1.27)
+				)
+			)
+		)
+		(property "Footprint" ""
+			(at 127 95.25 0)
+			(effects
+				(font
+					(size 1.27 1.27)
+				)
+				(hide yes)
+			)
+		)
+		(property "Datasheet" ""
+			(at 127 95.25 0)
+			(effects
+				(font
+					(size 1.27 1.27)
+				)
+				(hide yes)
+			)
+		)
+		(property "Description" "Power symbol creates a global label with name \"GND\" , ground"
+			(at 127 95.25 0)
+			(effects
+				(font
+					(size 1.27 1.27)
+				)
+				(hide yes)
+			)
+		)
+		(pin "1"
+		)
+		(instances
+			(project "Stern_pcb"
+				(path "/96f7660e-d3d9-4022-bb72-d6467b6cbc1f/33048040-4ae5-46e0-b14d-55f5f524b841"
+					(reference "#PWR045")
+					(unit 1)
+				)
+			)
+		)
+	)
+	(symbol
 		(lib_id "power:+12V")
 		(at 205.74 76.2 0)
@@
 					(unit 1)
 				)
+			)
+		)
+	)
+	(symbol
+		(lib_id "Device:R")
+		(at 127 90.17 0)
+		(unit 1)
+		(exclude_from_sim no)
+		(in_bom yes)
+		(on_board yes)
+		(dnp no)
+		(property "Reference" "R16"
+			(at 120.65 90.932 0)
+			(effects
+				(font
+					(size 1.27 1.27)
+				)
+				(justify left)
+			)
+		)
+		(property "Value" "10k"
+			(at 120.65 93.472 0)
+			(effects
+				(font
+					(size 1.27 1.27)
+				)
+				(justify left)
+			)
+		)
+		(property "Footprint" "Resistor_SMD:R_0603_1608Metric_Pad0.98x0.95mm_HandSolder"
+			(at 125.222 90.17 90)
+			(effects
+				(font
+					(size 1.27 1.27)
+				)
+				(hide yes)
+			)
+		)
+		(property "Datasheet" "~"
+			(at 127 90.17 0)
+			(effects
+				(font
+					(size 1.27 1.27)
+				)
+				(hide yes)
+			)
+		)
+		(property "Description" "Resistor"
+			(at 127 90.17 0)
+			(effects
+				(font
+					(size 1.27 1.27)
+				)
+				(hide yes)
+			)
+		)
+		(pin "2"
+		)
+		(pin "1"
+		)
+		(instances
+			(project "Stern_pcb"
+				(path "/96f7660e-d3d9-4022-bb72-d6467b6cbc1f/33048040-4ae5-46e0-b14d-55f5f524b841"
+					(reference "R16")
+					(unit 1)
+				)
