File: USB.kicad_sch (KiCad schematic)
At the start: 21 parts, among them J1 Conn_01x05, U3 BQ25895RTW

Commit message: assigned footprints
Parts:
- added J4: Conn_01x02, Connector_JST:JST_EH_B2B-EH-A_1x02_P2.50mm_Vertical, symbol Connector_Generic:Conn_01x02
- C13, C15, C2: footprint (none) -> Capacitor_SMD:C_0603_1608Metric_Pad1.08x0.95mm_HandSolder
- J1: footprint (none) -> Connector_JST:JST_PH_B5B-PH-K_1x05_P2.00mm_Vertical
- L2: footprint (none) -> Inductor_SMD:L_PSA_WLPMA0A040
- R2, R3: footprint (none) -> Resistor_SMD:R_0603_1608Metric_Pad0.98x0.95mm_HandSolder
- TH1: footprint (none) -> Connector_PinHeader_2.54mm:PinHeader_1x02_P2.54mm_Vertical
Connections:
- net +BATT: now also J4.1 (Pin_1)
- net D+: no longer J1.5 (Pin_5)
- net GND: now also J1.5 (Pin_5), J4.2 (Pin_2)
- net VSYS: now reaches C12.1, L2.2, U3.15 (SYS), U3.16 (SYS)

Commit message: Layout begonnen
Connections:
- net SW: now reaches C13.1, L2.1, U3.19 (SW), U3.20 (SW)
Changed lines of the file:
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@@
+		)
+	)
+	(label "SW"
+		(at 162.56 71.12 0)
+		(fields_autoplaced yes)
+		(effects
+			(font
+				(size 1.27 1.27)
+			)
+			(justify left bottom)
 		)
 	)

Commit message: marked unused capaacitors as not placed. Pull down on gate channel
Connections:
- net DSEL: no longer names the net of R10.2, U3.24 (DSEL)
Changed lines of the file:
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@@
-	)
-	(junction
-		(at 160.02 93.98)
-		(diameter 0)
-		(color 0 0 0 0)
 	)
 	(junction
@@
 		(pts
 			(xy 95.25 81.28) (xy 95.25 93.98)
-		)
-		(stroke
-			(width 0)
-			(type default)
-		)
-	)
-	(wire
-		(pts
-			(xy 160.02 93.98) (xy 163.83 93.98)
 		)
 		(stroke
@@
 				(hide yes)
 			)
-		)
-	)
-	(global_label "DSEL"
-		(shape input)
-		(at 163.83 93.98 0)
-		(fields_autoplaced yes)
-		(effects
-			(font
-				(size 1.27 1.27)
-			)
-			(justify left)
-		)
-		(property "Intersheetrefs" "${INTERSHEET_REFS}"
-			(at 171.4718 93.98 0)
-			(effects
-				(font
-					(size 1.27 1.27)
-				)
-				(justify left)
-				(hide yes)
-			)

Commit message: Verbindung zum Temperatursensor war falsch
Connections:
- net at R3.1, U3.11 (TS): now also R2.2, TH1.1; no longer R2.1
- net at C2.1, U3.22 (REGN): now also R2.1
Changed lines of the file:
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@@
+	)
+	(junction
+		(at 157.48 121.92)
+		(diameter 0)
+		(color 0 0 0 0)
+	)
+	(junction
+		(at 162.56 96.52)
+		(diameter 0)
+		(color 0 0 0 0)
 	)
 	(junction
@@
 	)
 	(junction
+		(at 167.64 121.92)
+		(diameter 0)
+		(color 0 0 0 0)
+	)
+	(junction
 		(at 190.5 46.99)
 		(diameter 0)
@@
 	(junction
 		(at 102.87 91.44)
-		(diameter 0)
-		(color 0 0 0 0)
-	)
-	(junction
-		(at 157.48 114.3)
 		(diameter 0)
 		(color 0 0 0 0)
@@
 	(wire
 		(pts
-			(xy 157.48 114.3) (xy 157.48 123.19)
+			(xy 157.48 101.6) (xy 157.48 121.92)
 		)
 		(stroke
@@
 	(wire
 		(pts
+			(xy 167.64 96.52) (xy 162.56 96.52)
+		)
+		(stroke
+			(width 0)
+			(type default)
+		)
+	)
+	(wire
+		(pts
 			(xy 59.69 77.47) (xy 59.69 74.93)
 		)
@@
 	(wire
 		(pts
+			(xy 167.64 114.3) (xy 167.64 96.52)
+		)
+		(stroke
+			(width 0)
+			(type default)
+		)
+	)
+	(wire
+		(pts
 			(xy 227.33 96.52) (xy 224.79 96.52)
 		)
@@
 	(wire
 		(pts
+			(xy 157.48 121.92) (xy 157.48 123.19)
+		)
+		(stroke
+			(width 0)
+			(type default)
+		)
+	)
+	(wire
+		(pts
 			(xy 134.62 52.07) (xy 134.62 66.04)
 		)
@@
 	(wire
 		(pts
-			(xy 157.48 114.3) (xy 157.48 101.6)
+			(xy 157.48 121.92) (xy 167.64 121.92)
 		)
 		(stroke
@@
 		)
 		(stroke
-			(width 0)
-			(type default)
-		)
-	)
-	(wire
-		(pts
-			(xy 157.48 114.3) (xy 167.64 114.3)
-		)
-		(stroke
